Commit message: Both robots now work!!!

File: catkin_botlers/src/gazebo_world/urdf/jackal.urdf.xacro (robot description, xacro)
@@ -1,4 +1,4 @@
 <?xml version="1.0"?>
-<robot name="combined" xmlns:xacro="http://www.ros.org/wiki/xacro">
+<robot name="jackal" xmlns:xacro="http://www.ros.org/wiki/xacro">
   <xacro:property name="PI" value="3.1415926535897931" />
   <xacro:property name="wheelbase" value="0.262" />
@@ -80,8 +80,8 @@
     <origin xyz="${-wheelbase/2} ${-track/2} ${wheel_vertical_offset}" rpy="0 0 0" />
   </xacro:wheel>
-  <link name="jackal_link"></link>
-  <joint name="jackal_link_joint" type="fixed">
+  <link name="base_link"></link>
+  <joint name="base_link_joint" type="fixed">
     <origin xyz="0 0 0" rpy="0 0 0" />
-    <parent link="jackal_link"/>
+    <parent link="base_link"/>
     <child link="chassis_link" />
   </joint>
@@ -219,22 +219,12 @@
   </joint>
   <!-- Bring in simulation data for Gazebo. -->
-  <xacro:include filename="$(find jackal_description)/urdf/jackal.gazebo" />
+  <xacro:include filename="$(find gazebo_world)/urdf/jackal.gazebo" />
   <!-- Optional standard accessories, including their simulation data. The rendering
        of these into the final description is controlled by optenv variables, which
        default each one to off.-->
   <xacro:include filename="$(find jackal_description)/urdf/accessories.urdf.xacro" />
-  <xacro:arg name="transmission_hw_interface" default="hardware_interface/PositionJointInterface"/>
-  <!-- common stuff -->
-  <xacro:include filename="$(find ur_description)/urdf/common.gazebo.xacro" />
-  <!-- ur3 -->
-  <!-- <xacro:include filename="$(find ur_description)/urdf/ur3.urdf.xacro"/> -->
-  <!-- arm -->
-  <!-- <xacro:ur3_robot prefix="" joint_limited="false"
-    transmission_hw_interface="$(arg transmission_hw_interface)"
-  /> -->
-  <!-- <joint name="connection_joint" type="fixed">
-    <parent link="mid_mount" />
-    <child link = "base_link" />
-    <origin xyz="0.0 0.0 0.0" rpy="0 0.0 3.14159265" />
-  </joint> -->
+  <!-- Optional custom includes. -->
+  <xacro:include filename="$(optenv JACKAL_URDF_EXTRAS empty.urdf)" />
+  <!-- Optional for Clearpath internal softwares -->
+  <xacro:include filename="$(optenv CPR_URDF_EXTRAS empty.urdf)" />
 </robot>
