Commit message: All changes, it works!!!

File: catkin_botlers/src/ur3/universal_robot/ur_description/urdf/ur3.urdf.xacro (robot description, xacro)
@@ -70,9 +70,9 @@
         </material>
       </visual>
-      <collision>
+      <!-- <collision>
         <geometry>
           <mesh filename="package://ur_description/meshes/ur3/collision/base.stl"/>
         </geometry>
-      </collision>
+      </collision> -->
       <xacro:cylinder_inertial radius="0.075" length="0.038" mass="${base_mass}">
         <origin xyz="0.0 0.0 0.0" rpy="0 0 0" />
@@ -107,9 +107,9 @@
         </material>
       </visual>
-      <collision>
+      <!-- <collision>
         <geometry>
           <mesh filename="package://ur_description/meshes/ur3/collision/shoulder.stl"/>
         </geometry>
-      </collision>
+      </collision> -->
       <xacro:cylinder_inertial radius="0.075" length="0.178" mass="${shoulder_mass}">
         <origin xyz="0.0 0.0 0.0" rpy="0 0 0" />
@@ -144,9 +144,9 @@
         </material>
       </visual>
-      <collision>
+      <!-- <collision>
         <geometry>
           <mesh filename="package://ur_description/meshes/ur3/collision/upperarm.stl"/>
         </geometry>
-      </collision>
+      </collision> -->
       <xacro:cylinder_inertial radius="0.075" length="${-a2}" mass="${upper_arm_mass}">
         <origin xyz="0.0 0.0 ${-a2/2.0}" rpy="0 0 0" />
@@ -181,9 +181,9 @@
         </material>
       </visual>
-      <collision>
+      <!-- <collision>
         <geometry>
           <mesh filename="package://ur_description/meshes/ur3/collision/forearm.stl"/>
         </geometry>
-      </collision>
+      </collision> -->
       <xacro:cylinder_inertial radius="0.075" length="${-a3}" mass="${forearm_mass}">
         <origin xyz="0.0 0.0 ${-a3/2.0}" rpy="0 0 0" />
@@ -218,9 +218,9 @@
         </material>
       </visual>
-      <collision>
+      <!-- <collision>
         <geometry>
           <mesh filename="package://ur_description/meshes/ur3/collision/wrist1.stl"/>
         </geometry>
-      </collision>
+      </collision> -->
       <xacro:cylinder_inertial radius="0.075" length="0.12" mass="${wrist_1_mass}">
         <origin xyz="0.0 ${wrist_1_length} 0.0" rpy="0 0 0" />
@@ -255,9 +255,9 @@
         </material>
       </visual>
-      <collision>
+      <!-- <collision>
         <geometry>
           <mesh filename="package://ur_description/meshes/ur3/collision/wrist2.stl"/>
         </geometry>
-      </collision>
+      </collision> -->
       <xacro:cylinder_inertial radius="0.075" length="0.12" mass="${wrist_2_mass}">
         <origin xyz="0.0 0.0 ${wrist_2_length}" rpy="0 0 0" />
@@ -292,9 +292,9 @@
         </material>
       </visual>
-      <collision>
+      <!-- <collision>
         <geometry>
           <mesh filename="package://ur_description/meshes/ur3/collision/wrist3.stl"/>
         </geometry>
-      </collision>
+      </collision> -->
       <xacro:cylinder_inertial radius="0.032" length="0.04" mass="${wrist_3_mass}">
         <origin xyz="0.0 ${wrist_3_length - 0.02} 0.0" rpy="${pi/2} 0 0" />
@@ -312,5 +312,5 @@
         </geometry>
       </visual>
-      <collision>
+      <!-- <collision>
         <geometry>
           <box size="0.01 0.01 0.01"/>
@@ -325,5 +325,5 @@
         </surface>
         <origin rpy="0 0 0" xyz="-0.01 0 0"/>
-      </collision>
+      </collision> -->
       <inertial>
         <origin rpy="0 0 0" xyz="0.000000 0.000000 0.000000"/>
